Commit message: Added toro example

File: model/toro/toro_original.urdf (robot description, URDF)
Before this commit: robot toro, 36 links, 35 joints
Links:
- removed link la_link7
- removed link ra_link7
Joints:
- removed joint j19_ee
- removed joint j25_ee

File: toro_example/toro.urdf (robot description, URDF)
Before this commit: robot toro, 36 links, 35 joints
Links:
- link la_link7: geometry visual box size=0.05 0.1 0.05; visual sphere radius=0.02
- link ra_link7: geometry visual box size=0.05 0.05 0.1; visual sphere radius=0.02
