Commit message: Fireone robot with two arms in starting position

File: Fireone/panda_arm.urdf (robot description, URDF)
Before this commit: robot panda, 15 links, 14 joints
Links:
- added link floating_virtual1, mass 1e-9
- added link floating_virtual2, mass 1e-9
- added link ground, mass 1e-9
- link linkbase: geometry visual mesh filename=../../../model/MobileBase/meshes/visual/Mobile_Base_03.obj
Joints:
- added joint floating_base_p1: type prismatic, parent ground, child floating_virtual1, origin xyz=0.000000 0.000000 0.000000 rpy=0.000000 0.000000 0.000000, axis 1 0 0, limit lower=-2.8973 upper=2.9873 effort=87 velocity=2.1750
- added joint floating_base_p2: type prismatic, parent floating_virtual1, child floating_virtual2, origin xyz=0.000000 0.000000 0.00000 rpy=0.000000 0.000000 0.000000, axis 0 1 0, limit lower=-2.8973 upper=2.9873 effort=87 velocity=2.1750
- added joint floating_base_r1: type revolute, parent floating_virtual2, child linkbase, origin xyz=0.000000 0.000000 0.00000 rpy=0.000000 0.000000 1.57079632679, axis 0 0 1, limit lower=-2.8973 upper=2.9873 effort=87 velocity=2.1750
- joint joint1: origin xyz=0 0.180389 0.83 rpy=0 0 0 -> xyz=0 0.180389 0.83 rpy=0 0 0.52359877559
- joint joint1r: origin xyz=0 -0.180389 0.83 rpy=0 0 -3.14159 -> xyz=0 -0.180389 0.83 rpy=0 0 -3.66519142919
- joint joint2: origin xyz=0 0 0 rpy=-1.57079632679 0 0 -> xyz=0 0 0 rpy=-1.57079632679 0.785000 0
- joint joint2r: origin xyz=0 0 0 rpy=-1.57079632679 0 0 -> xyz=0 0 0 rpy=-1.57079632679 -0.785000 0
- joint joint3: origin xyz=0 -0.316 0 rpy=1.57079632679 0 0 -> xyz=0 -0.316 0 rpy=1.57079632679 3.14159265359 0
- joint joint4: origin xyz=0.0825 0 0 rpy=1.57079632679 0 0 -> xyz=0.0825 0 0 rpy=1.57079632679 -0.52359877559 0
- joint joint4r: origin xyz=0.0825 0 0 rpy=1.57079632679 0 0 -> xyz=0.0825 0 0 rpy=1.57079632679 -0.52359877559 0
- joint joint5: origin xyz=-0.0825 0.384 0 rpy=-1.57079632679 0 0 -> xyz=-0.0825 0.384 0 rpy=-1.57079632679 -1.57079632679 0
- joint joint5r: origin xyz=-0.0825 0.384 0 rpy=-1.57079632679 0 0 -> xyz=-0.0825 0.384 0 rpy=-1.57079632679 -1.57079632679 0
- joint joint6: origin xyz=0 0 0 rpy=1.57079632679 0 0 -> xyz=0 0 0 rpy=1.57079632679 -1.0471975512 3.14159
- joint joint6r: origin xyz=0 0 0 rpy=1.57079632679 0 3.14159 -> xyz=0 0 0 rpy=1.57079632679 5.23598775598 0
- joint joint7: origin xyz=0.088 0 0 rpy=1.57079632679 0 0 -> xyz=0.088 0 0 rpy=1.57079632679 0.78539816339 0
- joint joint7r: origin xyz=0.088 0 0 rpy=1.57079632679 0 0 -> xyz=0.088 0 0 rpy=1.57079632679 0.78539816339 0

Commit message: arm movement and collision mesh uncommented. also commented base movement for now.

File: Fireone/panda_arm.urdf (robot description, URDF)
Before this commit: robot panda, 18 links, 17 joints
Links:
- link link1: geometry collision mesh filename=../../../model/panda/meshes/collision/link1.obj; visual mesh filename=../../../model/panda/meshes/visual/link1.obj
- link link1r: geometry collision mesh filename=../../../model/panda/meshes/collision/link1.obj; visual mesh filename=../../../model/panda/meshes/visual/link1.obj
- link link2: geometry collision mesh filename=../../../model/panda/meshes/collision/link2.obj; visual mesh filename=../../../model/panda/meshes/visual/link2.obj
- link link2r: geometry collision mesh filename=../../../model/panda/meshes/collision/link2.obj; visual mesh filename=../../../model/panda/meshes/visual/link2.obj
- link link3: geometry collision mesh filename=../../../model/panda/meshes/collision/link3.obj; visual mesh filename=../../../model/panda/meshes/visual/link3.obj
- link link3r: geometry collision mesh filename=../../../model/panda/meshes/collision/link3.obj; visual mesh filename=../../../model/panda/meshes/visual/link3.obj
- link link4: geometry collision mesh filename=../../../model/panda/meshes/collision/link4.obj; visual mesh filename=../../../model/panda/meshes/visual/link4.obj
- link link4r: geometry collision mesh filename=../../../model/panda/meshes/collision/link4.obj; visual mesh filename=../../../model/panda/meshes/visual/link4.obj
- link link5: geometry collision mesh filename=../../../model/panda/meshes/collision/link5.obj; visual mesh filename=../../../model/panda/meshes/visual/link5.obj
- link link5r: geometry collision mesh filename=../../../model/panda/meshes/collision/link5.obj; visual mesh filename=../../../model/panda/meshes/visual/link5.obj
- link link6: geometry collision mesh filename=../../../model/panda/meshes/collision/link6.obj; visual mesh filename=../../../model/panda/meshes/visual/link6.obj
- link link6r: geometry collision mesh filename=../../../model/panda/meshes/collision/link6.obj; visual mesh filename=../../../model/panda/meshes/visual/link6.obj
- link link7: geometry collision mesh filename=../../../model/panda/meshes/collision/link7.obj; visual mesh filename=../../../model/panda/meshes/visual/link7.obj
- link link7r: geometry collision mesh filename=../../../model/panda/meshes/collision/link7.obj; visual mesh filename=../../../model/panda/meshes/visual/link7.obj

Commit message: Adding potential field

File: Fireone/panda_arm.urdf (robot description, URDF)
Before this commit: robot panda, 18 links, 17 joints
Links:
- link link1: geometry visual mesh filename=../../../model/panda/meshes/visual/link1.obj
- link link1r: geometry visual mesh filename=../../../model/panda/meshes/visual/link1.obj
- link link2: geometry visual mesh filename=../../../model/panda/meshes/visual/link2.obj
- link link2r: geometry visual mesh filename=../../../model/panda/meshes/visual/link2.obj
- link link3: geometry visual mesh filename=../../../model/panda/meshes/visual/link3.obj
- link link3r: geometry visual mesh filename=../../../model/panda/meshes/visual/link3.obj
- link link4: geometry visual mesh filename=../../../model/panda/meshes/visual/link4.obj
- link link4r: geometry visual mesh filename=../../../model/panda/meshes/visual/link4.obj
- link link5: geometry visual mesh filename=../../../model/panda/meshes/visual/link5.obj
- link link5r: geometry visual mesh filename=../../../model/panda/meshes/visual/link5.obj
- link link6: geometry visual mesh filename=../../../model/panda/meshes/visual/link6.obj
- link link6r: geometry visual mesh filename=../../../model/panda/meshes/visual/link6.obj
- link link7: geometry visual mesh filename=../../../model/panda/meshes/visual/link7.obj; visual sphere radius=0.01
- link link7r: geometry visual mesh filename=../../../model/panda/meshes/visual/link7.obj; visual sphere radius=0.01
